File: KiCad/BardsAssistant/_autosave-BardsAssistant.kicad_pcb (KiCad board)
At the start: 2 copper layers, 100 x 100 mm, 75 parts, among them IC1 ESP32-S3-MINI-1-N8, J1 USB_C_Receptacle_USB2.0_16P, J2 Conn_01x24, J3 JST-PH-2-SMT-RA, Q1 Si1308EDL, Q3 AO3401A, SW1 SW_Push, SW2 SW_Push, SW3 SW_Push, SW4 SW_Push, SW5 SW_Push, SW6 SW_Push, U1 TPS63001, U2 USBLC6-2SC6, U3 MCP73831/2

Commit message: Added new KiCad revision
Parts:
- moved C10 7.30 mm to (155.0, 88.2)
- moved C17 7.30 mm to (159.4, 88.2)
- moved C22 7.30 mm to (163.9, 88.2)
- moved C5 7.30 mm to (150.7, 113.0)
- moved D5 7.30 mm to (132.2, 128.4)
- moved D6 7.30 mm to (168.4, 117.2)
- moved D9 7.30 mm to (169.2, 113.9)
- moved F1 7.30 mm to (127.9, 128.6)
- moved FB1 7.30 mm to (151.0, 128.2)
- moved J1 7.30 mm to (141.5, 109.5)
- moved R12 7.30 mm to (161.1, 124.4)
- moved R6 7.30 mm to (158.2, 124.4)
- moved R9 7.30 mm to (154.7, 113.0)
- moved SW4 7.30 mm to (130.0, 103.9)
- moved TP2 7.30 mm to (136.3, 120.3)
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Other:
- copper layers 2 -> 4
